File: rgbntsc.sch (KiCad schematic (older format))
At the start: 57 parts, among them J1 USB_C_Receptacle_Power, J2 VGA, J3 SCART_CONN, J4 Mini-DIN-4, U1 LM1881, U2 74AHCT1G86, U3 74AHCT1G86, U4 SC6206B-65K5, U5 CXA2075, U6 TPF144-VR, X1 O32253579545MHEA4SI

Commit message: ditched supply reg, just filter harder
Parts:
- removed R8: 1k, Resistor_SMD:R_0805_2012Metric, symbol rgbntsc-rescue:R_Small-Device
- removed R9: 1k5, Resistor_SMD:R_0805_2012Metric, symbol rgbntsc-rescue:R_Small-Device
- removed U4: SC6206B-65K5, Package_TO_SOT_SMD:SOT-23, symbol rgbntsc-rescue:MCP1700-2802E_SOT23-Regulator_Linear
- added FB2: Ferrite_Bead_Small, Capacitor_SMD:C_0805_2012Metric, symbol rgbntsc-rescue:Ferrite_Bead_Small-Device
- C12, C13, C14: symbol Device:CP_Small -> rgbntsc-rescue:CP_Small-Device
- D1: symbol Device:LED -> rgbntsc-rescue:LED-Device
- FB1: symbol Device:Ferrite_Bead_Small -> rgbntsc-rescue:Ferrite_Bead_Small-Device
- J1: symbol Videobits:USB_C_Receptacle_Power -> rgbntsc-rescue:USB_C_Receptacle_Power-Videobits
- J2: symbol ossc:VGA -> rgbntsc-rescue:VGA-ossc
- J3: symbol ossc:SCART_CONN -> rgbntsc-rescue:SCART_CONN-ossc
- U5: symbol Videobits:CXA2075 -> rgbntsc-rescue:CXA2075-Videobits
- U6: symbol Videobits:TPF144-VR -> rgbntsc-rescue:TPF144-VR-Videobits
Connections:
- net +5V: now also C9.1, FB2.1
- net VCC: now also FB2.2; no longer C9.1
Other:
- note removed: "1.8V really LDO"
- moved on the sheet: C9
Changed lines of the file:
@@
 $EndComp
-$Comp
-L rgbntsc-rescue:MCP1700-2802E_SOT23-Regulator_Linear U4
-U 1 1 5FA9BD42
-P 4800 6300
-F 0 "U4" H 4800 6542 50  0000 C CNN
-F 1 "SC6206B-65K5" H 4800 6451 50  0000 C CNN
-F 2 "Package_TO_SOT_SMD:SOT-23" H 4800 6525 50  0001 C CNN
-F 3 "http://ww1.microchip.com/downloads/en/DeviceDoc/20001826D.pdf" H 4800 6300 50  0001 C CNN
-F 4 "C88294" H 4800 6300 50  0001 C CNN "LCSC"
-	1    4800 6300
-	1    0    0    -1
-$EndComp
-$Comp
-L rgbntsc-rescue:R_Small-Device R8
-U 1 1 5FA9BD43
-P 5250 6450
-F 0 "R8" H 5309 6496 50  0000 L CNN
-F 1 "1k" H 5309 6405 50  0000 L CNN
-F 2 "Resistor_SMD:R_0805_2012Metric" H 5250 6450 50  0001 C CNN
-F 3 "~" H 5250 6450 50  0001 C CNN
-F 4 "C17513" H 5250 6450 50  0001 C CNN "LCSC"
-	1    5250 6450
-	1    0    0    -1
-$EndComp
-Wire Wire Line
-	5100 6300 5250 6300
-Wire Wire Line
-	5250 6300 5250 6350
-Wire Wire Line
-	5250 6550 5250 6600
-Wire Wire Line
-	4800 6600 5250 6600
-Connection ~ 5250 6600
-Connection ~ 5250 6300
-Wire Wire Line
-	5250 6600 5250 6650
-$Comp
-L rgbntsc-rescue:R_Small-Device R9
-U 1 1 5FA9BD44
-P 5250 6750
-F 0 "R9" H 5309 6796 50  0000 L CNN
-F 1 "1k5" H 5309 6705 50  0000 L CNN
-F 2 "Resistor_SMD:R_0805_2012Metric" H 5250 6750 50  0001 C CNN
-F 3 "~" H 5250 6750 50  0001 C CNN
-F 4 "C4310" H 5250 6750 50  0001 C CNN "LCSC"
-	1    5250 6750
-	1    0    0    -1
-$EndComp
-Wire Wire Line
-	5250 6850 5250 6900
-Connection ~ 5250 6900
 $Comp
 L rgbntsc-rescue:C_Small-Device C5
@@
 	1    0    0    -1
 $EndComp
-Text Notes 4500 6000 0    50   ~ 0
-1.8V really LDO
 Wire Wire Line
 	4600 1900 5050 1900
@@
 L rgbntsc-rescue:CP_Small-Device C9
 U 1 1 5CA25A7B
-P 5650 6600
-F 0 "C9" H 5738 6646 50  0000 L CNN
-F 1 "33u" H 5738 6555 50  0000 L CNN
-F 2 "Capacitor_SMD:CP_Elec_6.3x7.7" H 5650 6600 50  0001 C CNN
-F 3 "~" H 5650 6600 50  0001 C CNN
-F 4 "C127970" H 5650 6600 50  0001 C CNN "LCSC"
-	1    5650 6600
-	1    0    0    -1
-$EndComp
-Wire Wire Line
-	5650 6500 5650 6300
-Wire Wire Line
-	5650 6700 5650 6900
+P 4500 6600
+F 0 "C9" H 4588 6646 50  0000 L CNN
+F 1 "33u" H 4588 6555 50  0000 L CNN
+F 2 "Capacitor_SMD:CP_Elec_6.3x7.7" H 4500 6600 50  0001 C CNN
+F 3 "~" H 4500 6600 50  0001 C CNN
+F 4 "C127970" H 4500 6600 50  0001 C CNN "LCSC"
+	1    4500 6600
+	1    0    0    -1
+$EndComp
+Wire Wire Line
+	4500 6500 4500 6300
+Wire Wire Line
+	4500 6700 4500 6900
 Text Label 3850 1900 0    50   ~ 0
 Red
 $Comp
-L ossc:SCART_CONN J3
+L rgbntsc-rescue:SCART_CONN-ossc J3
 U 1 1 5FA9BD50
 P 2050 1500
@@
 	4400 2100 4400 2250
 $Comp
-L ossc:VGA J2
+L rgbntsc-rescue:VGA-ossc J2
 U 1 1 5CCA16CB
 P 2000 3200
@@
 $EndComp
 $Comp
-L converted:VCC #PWR07
+L rgbntsc-rescue:VCC-converted #PWR07
 U 1 1 5CCEB77D
 P 2700 4250
@@
 $EndComp
 $Comp
-L Videobits:USB_C_Receptacle_Power J1
+L rgbntsc-rescue:USB_C_Receptacle_Power-Videobits J1
 U 1 1 5FA9BD53
 P 1100 6150
@@
 Wire Wire Line
 	1450 4550 2200 4550
-Wire Wire Line
-	5250 6300 5650 6300
-Wire Wire Line
-	5250 6900 5650 6900
-Connection ~ 5650 6300
-Wire Wire Line
-	5650 6300 6050 6300
-Connection ~ 5650 6900
-Wire Wire Line
-	5650 6900 6050 6900
-Wire Wire Line
-	4050 6300 4500 6300
-Wire Wire Line
-	4050 6900 5250 6900
 $Comp
 L rgbntsc-rescue:Fiducial-Mechanical GOTE1
@@
 $EndComp
 $Comp
-L Videobits:CXA2075 U5
+L rgbntsc-rescue:CXA2075-Videobits U5
 U 1 1 5F8DCCCB
 P 7850 2000
@@
 	3000 3250 3000 3350
 $Comp
-L converted:VCC #PWR014
+L rgbntsc-rescue:VCC-converted #PWR014
 U 1 1 5FAA17A4
 P 3450 2950
@@
 $EndComp
 $Comp
-L converted:VCC #PWR09
+L rgbntsc-rescue:VCC-converted #PWR09
 U 1 1 5FAA17C4
 P 3000 3550
@@
 $EndComp
 $Comp
-L Device:CP_Small C14
+L rgbntsc-rescue:CP_Small-Device C14
 U 1 1 5FD38DD8
 P 9600 2100
@@
 $EndComp
 $Comp
-L Device:CP_Small C13
+L rgbntsc-rescue:CP_Small-Device C13
 U 1 1 5FD1A5C0
 P 9600 2000
@@
 $EndComp
 $Comp
-L Device:CP_Small C12
+L rgbntsc-rescue:CP_Small-Device C12
 U 1 1 5FD18E68
 P 9600 1900
@@
 	5050 2100 4800 2100
 $Comp
-L Videobits:TPF144-VR U6
+L rgbntsc-rescue:TPF144-VR-Videobits U6
 U 1 1 5FE6286C
 P 5450 2150
@@
 	7550 3350 7550 2400
 $Comp
-L Device:Ferrite_Bead_Small FB1
+L rgbntsc-rescue:Ferrite_Bead_Small-Device FB1
 U 1 1 60AAC928
 P 2100 5950
@@
 $EndComp
 $Comp
-L Device:LED D1
+L rgbntsc-rescue:LED-Device D1
 U 1 1 60C1D817
 P 6400 6750
@@
 Wire Wire Line
 	6400 6300 6050 6300
+Wire Wire Line
+	4050 6900 4500 6900
+Wire Wire Line
+	4050 6300 4500 6300
+Connection ~ 4500 6300
+Connection ~ 4500 6900
+Wire Wire Line
+	4500 6300 4950 6300
+Wire Wire Line
+	4500 6900 6050 6900
+$Comp
+L rgbntsc-rescue:Ferrite_Bead_Small-Device FB2
+U 1 1 61939B87
+P 5050 6300
+F 0 "FB2" V 5287 6300 50  0000 C CNN
+F 1 "Ferrite_Bead_Small" V 5196 6300 50  0000 C CNN
+F 2 "Capacitor_SMD:C_0805_2012Metric" V 4980 6300 50  0001 C CNN
+F 3 "~" H 5050 6300 50  0001 C CNN
+F 4 "C1017" V 5050 6300 50  0001 C CNN "LCSC"
+	1    5050 6300
+	0    -1   -1   0
+$EndComp
+Wire Wire Line
+	5150 6300 6050 6300
 $EndSCHEMATC

Commit message: swapping parts
Parts:
- removed U6: TPF144-VR, Package_SO:MSOP-10_3x3mm_P0.5mm, symbol rgbntsc-rescue:TPF144-VR-Videobits
- added U4: THS7374, Package_SO:TSSOP-14_4.4x5mm_P0.65mm, symbol Videobits:THS7374
- X1: value O32253579545MHEA4SI -> S7D3.579545A20F30T; footprint Oscillator:Oscillator_SMD_Abracon_ASE-4Pin_3.2x2.5mm -> Oscillator:Oscillator_SMD_Abracon_ASV-4Pin_7.0x5.1mm; LCSC C70606 -> C386914
Connections:
- net GND: now also U4.5 (Gnd), U4.6 (DIS), U4.9 (BYP)
- net VCC: now also U4.10 (Vcc)
- net at C5.1: now also U4.2 (In2)
- net at C6.1: now also U4.3 (In3)
- net at C7.1: now also U4.4 (In4)
- net at R20.2: now also U4.11 (Out4)
- net at R19.2: now also U4.12 (Out3)
- net at R18.2: now also U4.13 (Out2)
Changed lines of the file:
@@
 P 7100 4150
 F 0 "X1" H 7444 4196 50  0000 L CNN
-F 1 "O32253579545MHEA4SI" H 7444 4105 50  0000 L CNN
-F 2 "Oscillator:Oscillator_SMD_Abracon_ASE-4Pin_3.2x2.5mm" H 7800 3800 50  0001 C CNN
-F 3 "http://www.abracon.com/Oscillators/ASV.pdf" H 7000 4150 50  0001 C CNN
-F 4 "C70606" H 7100 4150 50  0001 C CNN "LCSC"
+F 1 "S7D3.579545A20F30T" H 7444 4105 50  0000 L CNN
+F 2 "Oscillator:Oscillator_SMD_Abracon_ASV-4Pin_7.0x5.1mm" H 7800 3800 50  0001 C CNN
+F 3 "https://datasheet.lcsc.com/lcsc/1912111437_Shenzhen-SCTF-Elec-S7D3-579545A20F30T_C386914.pdf" H 7000 4150 50  0001 C CNN
+F 4 "C386914" H 7100 4150 50  0001 C CNN "LCSC"
 	1    7100 4150
 	1    0    0    -1
@@
 	5050 2100 4800 2100
 $Comp
-L rgbntsc-rescue:TPF144-VR-Videobits U6
-U 1 1 5FE6286C
-P 5450 2150
-F 0 "U6" H 5475 3009 60  0000 C CNN
-F 1 "TPF144-VR" H 5475 2903 60  0000 C CNN
-F 2 "Package_SO:MSOP-10_3x3mm_P0.5mm" H 5475 2797 60  0000 C CNN
-F 3 "" H 5250 2400 60  0000 C CNN
-F 4 "C155447" H 5450 2150 50  0001 C CNN "LCSC"
-	1    5450 2150
-	1    0    0    -1
-$EndComp
-$Comp
-L rgbntsc-rescue:VCC-power #PWR0101
-U 1 1 5FE641C5
-P 5450 1600
-F 0 "#PWR0101" H 5450 1450 50  0001 C CNN
-F 1 "VCC" H 5467 1773 50  0000 C CNN
-F 2 "" H 5450 1600 50  0001 C CNN
-F 3 "" H 5450 1600 50  0001 C CNN
-	1    5450 1600
-	1    0    0    -1
-$EndComp
-$Comp
-L rgbntsc-rescue:GND-power #PWR0102
-U 1 1 5FE64C25
-P 5450 2600
-F 0 "#PWR0102" H 5450 2350 50  0001 C CNN
-F 1 "GND" H 5455 2427 50  0000 C CNN
-F 2 "" H 5450 2600 50  0001 C CNN
-F 3 "" H 5450 2600 50  0001 C CNN
-	1    5450 2600
-	1    0    0    -1
-$EndComp
-$Comp
 L rgbntsc-rescue:GND-power #PWR0103
 U 1 1 5FE6E447
@@
 Wire Wire Line
 	5150 6300 6050 6300
+$Comp
+L Videobits:THS7374 U4
+U 1 1 6272F820
+P 5250 1900
+F 0 "U4" H 5600 2250 60  0000 C CNN
+F 1 "THS7374" H 5750 2150 60  0000 C CNN
+F 2 "Package_SO:TSSOP-14_4.4x5mm_P0.65mm" H 5250 1900 60  0001 C CNN
+F 3 "" H 5250 1900 60  0000 C CNN
+	1    5250 1900
+	1    0    0    -1
+$EndComp
+$Comp
+L rgbntsc-rescue:GND-power #PWR038
+U 1 1 62730BCF
+P 5450 2600
+F 0 "#PWR038" H 5450 2350 50  0001 C CNN
+F 1 "GND" H 5455 2427 50  0000 C CNN
+F 2 "" H 5450 2600 50  0001 C CNN
+F 3 "" H 5450 2600 50  0001 C CNN
+	1    5450 2600
+	1    0    0    -1
+$EndComp
+$Comp
+L rgbntsc-rescue:VCC-converted #PWR037
+U 1 1 627316D0
+P 5450 1600
+F 0 "#PWR037" H 5450 1450 50  0001 C CNN
+F 1 "VCC" H 5465 1773 50  0000 C CNN
+F 2 "" H 5450 1600 60  0000 C CNN
+F 3 "" H 5450 1600 60  0000 C CNN
+	1    5450 1600
+	1    0    0    -1
+$EndComp
+$Comp
+L rgbntsc-rescue:GND-power #PWR039
+U 1 1 627365BF
+P 5900 2300
+F 0 "#PWR039" H 5900 2050 50  0001 C CNN
+F 1 "GND" H 5905 2127 50  0000 C CNN
+F 2 "" H 5900 2300 50  0001 C CNN
+F 3 "" H 5900 2300 50  0001 C CNN
+	1    5900 2300
+	0    -1   -1   0
+$EndComp
+$Comp
+L rgbntsc-rescue:GND-power #PWR036
+U 1 1 627371B6
+P 5050 2300
+F 0 "#PWR036" H 5050 2050 50  0001 C CNN
+F 1 "GND" H 5055 2127 50  0000 C CNN
+F 2 "" H 5050 2300 50  0001 C CNN
+F 3 "" H 5050 2300 50  0001 C CNN
+	1    5050 2300
+	0    1    1    0
+$EndComp
 $EndSCHEMATC
